Commit message: Update Camera and Lidar

File: description/camera.xacro (robot description, xacro)
@@ -2,29 +2,29 @@
 <robot xmlns:xacro="http://www.ros.org/wiki/xacro" >
     <joint name="camera_joint" type="fixed">
-        <parent link="chassis"/>
-        <child link="camera_link"/>
-        <origin xyz="0.276 0 0.181" rpy="0 0.18 0"/>
-    </joint>
-    <link name="camera_link">
-        <visual>
-            <geometry>
-                <box size="0.010 0.03 0.03"/>
-            </geometry>
-            <material name="black"/>
-        </visual>
-        <visual>
-            <origin xyz="0 0 -0.05"/>
-            <geometry>
-                <cylinder radius="0.002" length="0.1"/>
-            </geometry>
-            <material name="black"/>
-        </visual>
-    </link>
-    <joint name="camera_optical_joint" type="fixed">
-        <parent link="camera_link"/>
-        <child link="camera_link_optical"/>
-        <origin xyz="0 0 0" rpy="${-pi/2} 0 ${-pi/2}"/>
-    </joint>
-    <link name="camera_link_optical"></link>
+  <parent link="laser_frame"/>
+  <child link="camera_link"/>
+  <origin xyz="0 0 0.08" rpy="0 0 ${pi}"/> <!-- flipped to face forward -->
+</joint>
+<link name="camera_link">
+  <visual>
+    <geometry>
+      <box size="0.010 0.03 0.03"/>
+    </geometry>
+    <material name="black"/>
+  </visual>
+  <visual>
+    <origin xyz="0 0 -0.05"/>
+    <geometry>
+      <cylinder radius="0.002" length="0.1"/>
+    </geometry>
+    <material name="black"/>
+  </visual>
+</link>
+<joint name="camera_optical_joint" type="fixed">
+  <parent link="camera_link"/>
+  <child link="camera_link_optical"/>
+  <origin xyz="0 0 0" rpy="${-pi/2} 0 ${-pi/2}"/>
+</joint>
+<link name="camera_link_optical"/>
     <gazebo reference="camera_link">
         <material>Gazebo/Black</material>

File: description/lidar.xacro (robot description, xacro)
@@ -1,54 +1,70 @@
 <?xml version="1.0"?>
 <robot xmlns:xacro="http://www.ros.org/wiki/xacro" >
-    <joint name="laser_joint" type="fixed">
-        <parent link="chassis"/>
-        <child link="laser_frame"/>
-        <origin xyz="0.122 0 0.212" rpy="0 0 0"/>
-    </joint>
-    <link name="laser_frame">
-        <visual>
-            <geometry>
-                <cylinder radius="0.05" length="0.04"/>
-            </geometry>
-            <material name="black"/>
-        </visual>
-        <visual>
-            <origin xyz="0 0 -0.05"/>
-            <geometry>
-                <cylinder radius="0.01" length="0.1"/>
-            </geometry>
-            <material name="black"/>
-        </visual>
-        <collision>
-            <geometry>
-                <cylinder radius="0.05" length="0.04"/>
-            </geometry>
-        </collision>
-        <xacro:inertial_cylinder mass="0.1" length="0.04" radius="0.05">
-            <origin xyz="0 0 0" rpy="0 0 0"/>
-        </xacro:inertial_cylinder>
-    </link>
-    <gazebo reference="laser_frame">
-        <material>Gazebo/Black</material>
-        <sensor name="laser" type="gpu_lidar">
-            <pose> 0 0 0 0 0 0 </pose>
-            <visualize>false</visualize>
-            <update_rate>10</update_rate>
-            <lidar>
-                <scan>
-                    <horizontal>
-                        <samples>360</samples>
-                        <min_angle>-3.14</min_angle>
-                        <max_angle>3.14</max_angle>
-                    </horizontal>
-                </scan>
-                <range>
-                    <min>0.3</min>
-                    <max>12</max>
-                </range>
-            </lidar>
-            <topic>scan</topic>
-            <gz_frame_id>laser_frame</gz_frame_id>
-        </sensor>
-    </gazebo>
+  <!-- Turret link that raises the lidar -->
+  <joint name="lidar_turret_joint" type="fixed">
+    <parent link="chassis"/>
+    <child link="lidar_turret"/>
+    <origin xyz="0.122 0 0.10" rpy="0 0 0"/>
+  </joint>
+<link name="lidar_turret">
+  <visual>
+    <geometry>
+      <cylinder radius="0.04" length="0.5"/>
+    </geometry>
+    <material name="black"/>
+  </visual>
+  <collision>
+    <geometry>
+      <cylinder radius="0.04" length="0.08"/>
+    </geometry>
+  </collision>
+  <xacro:inertial_cylinder mass="0.05" length="0.08" radius="0.04">
+    <origin xyz="0 0 0" rpy="0 0 0"/>
+  </xacro:inertial_cylinder>
+</link>
+  <!-- LiDAR now mounted on turret -->
+<joint name="laser_joint" type="fixed">
+  <parent link="lidar_turret"/>
+  <child link="laser_frame"/>
+  <origin xyz="0 0 0.05" rpy="0 0 0"/> <!-- height adjusted -->
+</joint>
+  <link name="laser_frame">
+    <visual>
+      <geometry>
+        <cylinder radius="0.05" length="0.04"/>
+      </geometry>
+      <material name="black"/>
+    </visual>
+    <collision>
+      <geometry>
+        <cylinder radius="0.05" length="0.04"/>
+      </geometry>
+    </collision>
+    <xacro:inertial_cylinder mass="0.1" length="0.04" radius="0.05">
+      <origin xyz="0 0 0" rpy="0 0 0"/>
+    </xacro:inertial_cylinder>
+  </link>
+  <gazebo reference="laser_frame">
+    <material>Gazebo/Black</material>
+    <sensor name="laser" type="gpu_lidar">
+      <pose>0 0 0 0 0 0</pose>
+      <visualize>true</visualize>
+      <update_rate>10</update_rate>
+      <lidar>
+        <scan>
+          <horizontal>
+            <samples>360</samples>
+            <min_angle>-3.14</min_angle>
+            <max_angle>3.14</max_angle>
+          </horizontal>
+        </scan>
+        <range>
+          <min>0.3</min>
+          <max>12</max>
+        </range>
+      </lidar>
+      <topic>scan</topic>
+      <gz_frame_id>laser_frame</gz_frame_id>
+    </sensor>
+  </gazebo>
 </robot>
