Commit message: Adding simple robot arm

File: description/robot.urdf.xacro (robot description, xacro)
@@ -14,3 +14,4 @@
     <!-- <xacro:include filename="depth_camera.xacro" /> -->
     <xacro:include filename="face.xacro" />
+    <xacro:include filename="robot_arm.xacro" />
 </robot>

File: description/robot_core.xacro (robot description, xacro)
@@ -175,3 +175,8 @@
     <mu2 value="0.001"/>
   </gazebo>
+<joint name="robot_arm_mount" type="fixed">
+  <parent link="base_link"/>
+  <child link="arm_base"/>
+  <origin xyz="0.0 0.0 0.3" rpy="0 0 0"/>
+</joint>
 </robot>

Commit message: Removed identifier files

File: description/robot.urdf.xacro (robot description, xacro)
@@ -15,3 +15,8 @@
     <xacro:include filename="face.xacro" />
     <xacro:include filename="robot_arm.xacro" />
+    <joint name="robot_arm_mount" type="fixed">
+    <parent link="base_link"/>
+    <child link="arm_base"/>
+    <origin xyz="0.0 0.0 1.0" rpy="0 0 0"/>
+    </joint>
 </robot>

File: description/robot_arm.xacro (robot description, xacro)
@@ -105,10 +105,4 @@
   </link>
   <!-- ===================== JOINTS ===================== -->
-  <joint name="arm_base_joint" type="continuous">
-    <parent link="base_link"/> <!-- Attach externally -->
-    <child link="arm_base"/>
-    <origin xyz="0 0 0.3" rpy="0 0 0"/>
-    <axis xyz="0 0 1"/>
-  </joint>
   <joint name="shoulder_joint" type="continuous">
     <parent link="arm_base"/>

File: description/robot_core.xacro (robot description, xacro)
@@ -175,8 +175,3 @@
     <mu2 value="0.001"/>
   </gazebo>
-<joint name="robot_arm_mount" type="fixed">
-  <parent link="base_link"/>
-  <child link="arm_base"/>
-  <origin xyz="0.0 0.0 0.3" rpy="0 0 0"/>
-</joint>
 </robot>
